File: esp32-stick.kicad_sch (KiCad schematic)
At the start: 18 parts, among them Q1 BSS138, Q2 BSS138, SW1 SW_Push, SW2 SW_Push, U1 ESP32-WROOM-32, U2 AMS1117-3.3, U3 CH340C

Commit message: add pcb
Parts:
- removed U3: CH340C, CH340C:SO016, symbol CH340C:CH340C
- added J1: USB_A, Connector_USB:USB_A_CNCTech_1001-011-01101_Horizontal, symbol Connector:USB_A
- added U4: CH340C, Package_SO:SOIC-16_3.9x9.9mm_P1.27mm, symbol Interface_USB:CH340C
Connections:
- net +3V3: now also U4.16 (VCC), U4.4 (V3)
- net +5V: now also J1.1 (VBUS)
- net D+: now also J1.3 (D+), U4.5 (UD+)
- net D-: now also J1.2 (D-), U4.6 (UD-)
- net GND: now also J1.4 (GND), U4.1 (GND)
- net RX-PROG: now also U4.3 (RXD)
- net TX-PROG: now also U4.2 (TXD)
- net at Q1.2 (S), Q2.1 (G): now also U4.14 (~{RTS})
- net at Q1.1 (G), Q2.2 (S): now also U4.13 (~{DTR})
Other:
- moved on the sheet: C4

Commit message: board wiring
Parts:
- renumbered SW2 to BOOT, SW1 to EN
Changed lines of the file:
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@@
   (symbol (lib_id "Switch:SW_Push") (at 26.67 64.77 0) (unit 1)
     (in_bom yes) (on_board yes) (dnp no) (fields_autoplaced)
-    (property "Reference" "SW1" (at 26.67 57.15 0)
+    (property "Reference" "EN" (at 26.67 57.15 0)
       (effects (font (size 1.27 1.27)))
     )
@@
       (project "esp32-stick"
         (path "/7436125a-2c6b-4389-8bb5-11a61c536837"
-          (reference "SW1") (unit 1)
+          (reference "EN") (unit 1)
         )
       )
@@
   (symbol (lib_id "Switch:SW_Push") (at 88.9 64.77 0) (unit 1)
     (in_bom yes) (on_board yes) (dnp no) (fields_autoplaced)
-    (property "Reference" "SW2" (at 88.9 57.15 0)
+    (property "Reference" "BOOT" (at 88.9 57.15 0)
       (effects (font (size 1.27 1.27)))
     )
@@
       (project "esp32-stick"
         (path "/7436125a-2c6b-4389-8bb5-11a61c536837"
-          (reference "SW2") (unit 1)
-        )
-      )
+          (reference "BOOT") (unit 1)
+        )
+      )
