File: esp32-stick.kicad_pcb (KiCad board)
At the start: 2 copper layers, 48 x 25 mm, 19 parts, among them J1 USB_A, Q1 BSS138, Q2 BSS138, U1 ESP32-WROOM-32, U2 AMS1117-3.3, U4 CH340C

Commit message: wiring + fill zone
Parts:
- moved C4 36.4 mm to (74.0, 81.7)
- moved C2 34.4 mm to (75.6, 81.7)
Routing:
- net ESP32_EN: track 15.9 -> 47.4 mm, vias 0 -> 2
- net ESP32_IO0: track 10.1 -> 22.2 mm
- net +3V3: track 79.9 -> 76.9 mm
- net GND: vias 0 -> 8
- added copper zone on B.Cu, net GND
- added copper zone on F.Cu, net GND
Other:
- outline, holes or cut-outs redrawn
